File: Actuator_Controller_2026/Actuator_Controller_2026.kicad_sch (KiCad schematic)
At the start: 11 parts, among them J1 Conn_01x02_Pin, U2 L7815, U3 LMD18200, U4 LMD18200

Commit message: Finished actuator controller schematic
Changes to add:
Change the voltage regualtor
Remove the arduino and add screw terminals
Parts:
- added C10, C12: 100uF, project_footprints:CPolarized_Axial_L3.8mm_D2.6mm_P7.50mm_Horizontal, symbol project_symbols:C_Polarized
- added C11, C9: 1uF, project_footprints:CPolarized_Axial_L3.8mm_D2.6mm_P7.50mm_Horizontal, symbol project_symbols:C_Polarized
- added C13, C14, C7, C8: 10 nF, project_footprints:C_Axial_L3.8mm_D2.6mm_P7.50mm_Horizontal, symbol project_symbols:C
- added J2, J3, J4, J5: Screw_Terminal_01x04, symbol Connector:Screw_Terminal_01x04
- added J7, J8: Screw_Terminal_01x02, symbol Connector:Screw_Terminal_01x02
- added R5, R6: 10k, Resistor_THT:R_Box_L13.0mm_W4.0mm_P9.00mm, symbol Device:R
Connections:
- net M1_BOOT1: now reaches U3.1 (BOOTSTRAP1)
- net M1_BOOT1: now also C7.2
- net at U3.10 (OUTPUT2): now also C8.2, J2.3 (Pin_3), J2.4 (Pin_4)
- net M1_BOOT2: now reaches U3.11 (BOOTSTRAP2)
- net M1_BOOT2: now also C8.1
- net at U3.2 (OUTPUT1): now also C7.1, J2.1 (Pin_1), J2.2 (Pin_2)
- net M1_DIR: now reaches U3.3 (DIRECTION)
- net M1_DIR: now also A1.23 (D8)
- net GND: now reaches U3.4 (BRAKE)
- net GND: now also A1.29 (GND), A1.6 (GND), A1.7 (GND), U3.7 (GND), U4.4 (BRAKE), U4.7 (GND), C10.2, C11.2, C12.2, C9.2
- net M1_PWM: now reaches U3.5 (PWM)
- net M1_PWM: now also A1.24 (D9)
- net +15V: now reaches U3.6 (VS)
- net +15V: now also U4.6 (VS), C10.1, C11.1, C12.1, C9.1
- net M1_CFLAG: now reaches U3.8 (CURRENT_SENSE_OUTPUT)
- net M1_CFLAG: now also A1.26 (D11), J3.1 (Pin_1), J3.2 (Pin_2)
- net M1_TFLAG: now reaches U3.9 (~{THERMAL_FLAG_OUTPUT})
- net M1_TFLAG: now also A1.20 (D5), J3.3 (Pin_3), J3.4 (Pin_4), R5.2
- net M2_HALL: now reaches A1.18 (D3)
- net M2_HALL: now also J8.1 (Pin_1), J8.2 (Pin_2)
- net M1_HALL: now reaches A1.19 (D4)
- net M1_HALL: now also J7.1 (Pin_1), J7.2 (Pin_2)
- net M2_TFLAG: now reaches A1.21 (D6)
- net M2_TFLAG: now also U4.9 (~{THERMAL_FLAG_OUTPUT}), J5.3 (Pin_3), J5.4 (Pin_4), R6.2
- net M2_DIR: now reaches A1.22 (D7)
- net M2_DIR: now also U4.3 (DIRECTION)
- net M2_PWM: now reaches A1.25 (D10)
- net M2_PWM: now also U4.5 (PWM)
- net M2_CFLAG: now reaches A1.27 (D12)
- net M2_CFLAG: now also U4.8 (CURRENT_SENSE_OUTPUT), J5.1 (Pin_1), J5.2 (Pin_2)
- net M2_BOOT1: now reaches U4.1 (BOOTSTRAP1)
- net M2_BOOT1: now also C13.2
- net at U4.10 (OUTPUT2): now also C14.2, J4.3 (Pin_3), J4.4 (Pin_4)
- net M2_BOOT2: now reaches U4.11 (BOOTSTRAP2)
- net M2_BOOT2: now also C14.1
- net at U4.2 (OUTPUT1): now also C13.1, J4.1 (Pin_1), J4.2 (Pin_2)
- new net +5V: R5.1, R6.1
Other:
- note added: "*377 μA/A"
- note added: "DS suggests 100uF per amp output"
- moved on the sheet: A1, C1, C2, DZ1, J1, TP1, TP2, TP3, U2, U3
